File: KiCAD/rasPower-ILI9341_TFT_Touch_Screen/rasPower-ILI9341_TFT_Touch_Screen.kicad_sch (KiCad schematic)
At the start: 2 parts, among them J1 Raspberry_Pi_2_3, U2 ST7735_1.8"_TFT_128x160_w_SD-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

Commit message: new pin
Connections:
- net at J1.16 (GPIO23): no longer U2.5 (A0)
- net at J1.22 (GPIO25): now also U2.5 (A0)
Changed lines of the file:
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@@
-	(wire
-		(pts
-			(xy 66.04 102.87) (xy 83.82 102.87)
-		)
-		(stroke
-			(width 0)
-			(type default)
-		)
-	)
 	(wire
 		(pts
@@
 	(wire
 		(pts
+			(xy 83.82 107.95) (xy 66.04 107.95)
+		)
+		(stroke
+			(width 0)
+			(type default)
+		)
+	)
+	(wire
+		(pts
 			(xy 146.05 90.17) (xy 146.05 100.33)
 		)
@@
 	(wire
 		(pts
-			(xy 66.04 154.94) (xy 66.04 102.87)
-		)
-		(stroke
-			(width 0)
-			(type default)
-		)
-	)
-	(wire
-		(pts
 			(xy 161.29 85.09) (xy 161.29 52.07)
 		)
@@
 		)
 		(stroke
+			(width 0)
+			(type default)
+		)
+	)
+	(wire
+		(pts
+			(xy 66.04 107.95) (xy 66.04 154.94)
+		)
+		(stroke
